File: smart_relay.kicad_sch (KiCad schematic)
At the start: 8 parts, among them J2 Screw_Terminal_01x04, U1 BP8005

Commit message: Auto commit: 2025-03-07_01-56
Parts:
- removed D4: D, symbol Device:D
- removed J2: Screw_Terminal_01x04, TerminalBlock:TerminalBlock_MaiXu_MX126-5.0-04P_1x04_P5.00mm, symbol Connector:Screw_Terminal_01x04
- removed R: R10, symbol Device:R
- removed R1: R11, symbol Device:R
- removed RV1: R_Variable, 3225-471H:Untitled, symbol Device:R_Variable
- added C1, C29, C3, C30, C4, C5, C6, C8: C, symbol Device:C
- added C1, CE3, CE5: C_Polarized, symbol Device:C_Polarized
- added D1, D2, D3, D7, D9: F7, symbol Device:D
- added D2: UM10B, Package_TO_SOT_SMD:TO-269AA, symbol Diode_Bridge:RMB4S
- added D3: T4, symbol Device:D
- added D8: S120 / 2389, symbol Device:D
- added D9: TVS1, symbol Device:D
- added DZ1: D_Zener, symbol Device:D_Zener
- added Q1: NMOS, symbol Simulation_SPICE:NMOS
- added R1: R_Variable, symbol Device:R_Variable
- added R11, R13, R20, R21 (x2), R28, R30, R4, R7: R, symbol Device:R
- added R29: 10, symbol Device:R
- added R3: 1k, symbol Device:R
- added R8: 39, symbol Device:R
- added T1: EE8.3, symbol transformer_integrated_inductor:EE8.3
- added U2: OR-357 C, Package_DIP:DIP-4_W7.62mm, symbol Isolator:SFH617A-1
- added U3: BP2535C, symbol BP8005:BP2535C
- added U4: ME6231/3v3, Package_TO_SOT_SMD:SOT-223-3_TabPin2, symbol Regulator_Linear:AMS1117-3.3
- U1: footprint BP8005:SOT33-5B_L3.9-W2.6-P0.90-LS4.0-BL -> (none)
Connections:
- net at U1.1 (VIN): now also C5.2, D3.1 (K), D9.1 (K)
- net at U1.2 (FB2): now also C1.2, R4.2, R7.1
- net at R12.1, U1.3 (GATE): now also R11.2
- net GND: now reaches U1.4 (GND)
- net GND: now also C1.1, C29.1, C3.1, C30.1, C4.2, C5.1, C6.1, CE3.2, CE5.2, D2.2, D9.2 (A), DZ1.2 (A), Q1.3 (S), R1.2, R13.2, R7.2, T1.6 (1), U4.1 (GND)
- net at U1.5 (RST): now also R28.1
- net GNDREF: now reaches C2.1
- net GNDREF: now also C1.2, C4.1, C8.1, D2.4 (-), R21.2, R21.2, T1.4
- net at R12.2: now also D3.1 (K)
- net mosfet_gate: no longer names the net of C2.2
- net mosfet_gate: now also R21.1, U2.3, U3.2 (FB)
- new net: D2.1, R1.1, R8.1
- new net: D2.2 (A), D3.2 (A), D9.1 (K), Q1.1 (D), R4.1
- new net: DZ1.1 (K), R20.2, U2.2
- new net: CE3.1, D1.1 (K), D2.1 (K), U4.2 (VI)
- new net: C1.1, R3.1, T1.3 (6)
- new net: D2.3 (+), R3.2
- new net: D8.2 (A), T1.5 (2)
- new net: C8.2, D7.1 (K), U2.4, U3.3 (VCC)
- new net: D7.2 (A), R29.1
- new net: R20.1, R30.2, U2.1
- new net: R21.1, U3.5 (CS)
- new net: T1.2 (5), U3.4 (DRAIN)
- new net: R29.2, T1.1 (3)
- new net +3V3: C29.2, C30.2, C6.2, U4.3 (VO)
- new net +5V5: CE5.1, D1.2 (A), D8.1 (K), D9.2 (A), R30.1
- new net GATE: C3.2, D3.2 (A), Q1.2 (G), R11.1, R13.1
- new net L_OUT: R8.2
- new net rst_mcu: R28.2

Commit message: Auto commit: 2025-03-08_02-13
Parts:
- added C9: C, Capacitor_SMD:C_0402_1005Metric, symbol Device:C
- added D5: A7, Diode_SMD:D_SOD-123, symbol Device:D
- added ESD1: CC, Diode_SMD:D_SOD-323, symbol Device:D
- added J1: Screw_Terminal_01x04, TerminalBlock:TerminalBlock_MaiXu_MX126-5.0-04P_1x04_P5.00mm, symbol Connector:Screw_Terminal_01x04
- added Q4: SS8550, Package_TO_SOT_SMD:SOT-23, symbol Transistor_BJT:SS8550
- added Q5: SS8050, Package_TO_SOT_SMD:SOT-23, symbol Transistor_BJT:SS8050
- added R14, R18, R19, R22, R31: 0, Resistor_SMD:R_0402_1005Metric, symbol Device:R
- added R9: 75k, Resistor_SMD:R_1206_3216Metric, symbol Device:R
- C1, C30: footprint (none) -> Capacitor_SMD:C_0402_1005Metric
- C10: renamed from C5; footprint (none) -> Capacitor_SMD:C_1206_3216Metric
- C2: renamed from C3; footprint (none) -> Capacitor_SMD:C_0402_1005Metric
- C29, C6: footprint (none) -> Capacitor_SMD:C_0603_1608Metric
- C3: renamed from C1; value C_Polarized -> 1u/400v; footprint (none) -> Capacitor_SMD:CP_Elec_5x5.3
- C4: footprint (none) -> Capacitor_SMD:C_1206_3216Metric
- C5: renamed from C2; value C -> 100p; footprint (none) -> Capacitor_SMD:C_0402_1005Metric
- C8: footprint (none) -> Capacitor_SMD:C_0805_2012Metric
- CE3: value C_Polarized -> 680u/10v; footprint (none) -> Capacitor_THT:CP_Radial_D6.3mm_P2.50mm
- CE5: value C_Polarized -> 220u/10v; footprint (none) -> Capacitor_THT:CP_Radial_D5.0mm_P2.50mm
- D1, D2, D3, D7, D8, D9, DZ1: footprint (none) -> Diode_SMD:D_SOD-123
- D4: renamed from D3; footprint (none) -> Diode_SMD:D_SOD-323
- DB1: renamed from D2; footprint Package_TO_SOT_SMD:TO-269AA -> UM10B:UMB-4_L3.8-W3.6-P2.50-LS4.9-BL
- Q3: renamed from Q1; value NMOS -> AGM402A1; footprint (none) -> AGM402A1:DFN-8_L5.8-W4.9-P1.27-LS6.0-BL-1
- R10: renamed from R11; footprint (none) -> Resistor_SMD:R_0402_1005Metric
- R11: renamed from R13; footprint (none) -> Resistor_SMD:R_0402_1005Metric
- R12, R20, R21, R28, R4, R7: footprint (none) -> Resistor_SMD:R_0402_1005Metric
- R16: renamed from R21; footprint (none) -> Resistor_SMD:R_0805_2012Metric
- R29: footprint (none) -> Resistor_SMD:R_0805_2012Metric
- R3: footprint (none) -> Resistor_SMD:R_1210_3225Metric
- R30: footprint (none) -> Resistor_SMD:R_0603_1608Metric
- R8: footprint (none) -> Resistor_THT:R_Axial_DIN0207_L6.3mm_D2.5mm_P5.08mm_Vertical
- RV1: renamed from R1; footprint (none) -> 3225-471H:Untitled
- T1: footprint (none) -> Transformer:EE8.3
- TVS1: renamed from D9; footprint (none) -> Diode_SMD:D_1206_3216Metric
- U1: footprint (none) -> BP8005:SOT33-5B_L3.9-W2.6-P0.90-LS4.0-BL
- U2: footprint Package_DIP:DIP-4_W7.62mm -> OR357:SOP-4_L4.4-W3.9-P2.54-LS7.0-BL
- U3: footprint (none) -> BP2535C:SOT33-5A_L3.9-W2.6-P0.90-BP2525D
- U4: footprint Package_TO_SOT_SMD:SOT-223-3_TabPin2 -> ME6231A33:SOT-89-3_L4.5-W2.5-P1.50-LS4.2-BR
Connections:
- net +3V3: now also Q4.2 (E), R19.1, R22.2
- net GND: now also DB1.1, Q3.1 (S), C9.1, ESD1.1 (K), J1.2 (Pin_2), J1.3 (Pin_3), Q5.2 (E), R18.2; no longer DB1.2, Q3.3 (S)
- net GNDREF: now also U3.1 (GND)
- net L_OUT: now also J1.4 (Pin_4)
- net at R8.1, RV1.1: now also DB1.2; no longer DB1.1
- net at D2.2 (A), D3.2 (A), R4.1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: now also Q3.3 (D); no longer Q3.1 (D)
- net +5V5 renamed VBUS
- net GATE: no longer names the net of C2.2, D4.2 (A), Q3.2 (G), R10.1, R11.1
- new net: C9.2, ESD1.2 (A), R22.1, R31.1, R9.2
- new net: D5.2 (A), R9.1
- new net: Q4.3 (C), R14.1, R18.1
- new net: Q4.1 (B), R31.2
- new net: Q5.1 (B), R14.2
- new net MCU_Sw: Q5.3 (C), R19.2
- new net S2: D5.1 (K), J1.1 (Pin_1)
Other:
- moved on the sheet: DB1

Commit message: Auto commit: 2025-03-11_00-25
Parts:
- R30: value R -> 100
Connections:
- net GND: now also ESD1.2 (A); no longer ESD1.1 (K)
- net at C9.2, R22.1, R31.1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: now also ESD1.1 (K); no longer ESD1.2 (A)
Other:
- moved on the sheet: ESD1
Changed lines of the file:
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@@
 	(symbol
 		(lib_id "Device:D")
-		(at 403.86 217.17 90)
+		(at 403.86 217.17 270)
 		(unit 1)
 		(exclude_from_sim no)
@@
 					(size 1.27 1.27)
 				)
-				(justify right)
+				(justify left)
 			)
 		)
@@
 					(size 1.27 1.27)
 				)
-				(justify right)
+				(justify left)
 			)
 		)
@@
 			)
 		)
-		(property "Value" "R"
+		(property "Value" "100"
 			(at 259.08 73.6599 0)
 			(effects
