File: relay/relay/relay.kicad_sch (KiCad schematic)
At the start: 3 parts, among them K1 HFE60P/12-1HST-L2

Commit message: Auto commit: 2025-03-27_21-00
Parts:
- added C1, C2: C, symbol Device:C
- added Q1, Q2: SS8050, Package_TO_SOT_SMD:SOT-23, symbol Transistor_BJT:SS8050
- added R1, R2, R3, R4: R, symbol Device:R
- added R5: 0, symbol Device:R
Connections:
- net at D1.1 (K), K1.1: now also D2.1 (K), K1.3, C1.1, C2.1, R5.2
- net at K1.2: now also D2.2 (A), Q1.3 (C)
- net at K1.4: now also D1.2 (A), Q2.3 (C)
- new net: Q2.1 (B), R1.1, R4.1
- new net: Q1.1 (B), R2.1, R3.2
- new net 3v3: R5.1
- new net GND: C1.2, C2.2, Q1.2 (E), Q2.2 (E), R1.2, R2.2
- new net RESET: R4.2
- new net SET: R3.1
Other:
- moved on the sheet: D1, D2, K1
